File: kicad/horno.kicad_pcb (KiCad board)
At the start: 2 copper layers, 100.1 x 100.1 mm, 51 parts, among them P1 LPC1769, P10 Alimentación, P3 Termocupla, P4 TRIAC, P5 24V, P6 Motor, P7 Pantalla, P8 UART, P9 GPIO, Q1 BC547, SW1 RST, U1 OP07, U2 OP07, U3 LTC1050, U4 OP07, U5 L293D, U6 LM35

Commit message: últimas modificaciones al impreso.
Connections:
- P1 pad 11: /LPC1769/GPIO9 -> /LPC1769/GPIO14
- P1 pad 12: /LPC1769/GPIO8 -> /LPC1769/GPIO13
- P1 pad 13: /LPC1769/GPIO7 -> /LPC1769/GPIO12
- P1 pad 14: Net-(P1-Pad14) -> /LPC1769/GPIO11
- P1 pad 16: Net-(P1-Pad16) -> /LPC1769/GPIO10
- P1 pad 17: /LPC1769/GPIO6 -> /LPC1769/GPIO9
- P1 pad 18: /LPC1769/GPIO5 -> /LPC1769/GPIO8
- P1 pad 19: /LPC1769/GPIO4 -> /LPC1769/GPIO7
- P1 pad 20: Net-(P1-Pad20) -> /LPC1769/GPIO6
- P1 pad 21: Net-(P1-Pad21) -> /LPC1769/GPIO5
- P1 pad 23: Net-(P1-Pad23) -> /LPC1769/GPIO4
- P1 pad 5: /LPC1769/GPIO13 -> /LPC1769/GPIO18
- P1 pad 6: /LPC1769/GPIO12 -> /LPC1769/GPIO17
- P1 pad 7: /LPC1769/GPIO11 -> /LPC1769/GPIO16
- P1 pad 8: /LPC1769/GPIO10 -> /LPC1769/GPIO15
- P9 pad 17: Net-(P9-Pad17) -> /LPC1769/GPIO14
- P9 pad 18: +5V -> /LPC1769/GPIO15
- P9 pad 19: Net-(P9-Pad19) -> /LPC1769/GPIO16
- P9 pad 20: +5V -> /LPC1769/GPIO17
- P9 pad 21: GNDD -> /LPC1769/GPIO18
- P9 pad 22: GNDD -> +5V
Routing:
- net /LPC1769/GPIO14: track 0.00 -> 70.4 mm
- net /LPC1769/GPIO15: track 0.00 -> 56.8 mm
- net /LPC1769/GPIO16: track 0.00 -> 54.2 mm
- net /LPC1769/GPIO17: track 0.00 -> 45.7 mm
- net /LPC1769/GPIO18: track 0.00 -> 43.4 mm
- net /LPC1769/GPIO10: track 66.3 -> 94.8 mm
- net /LPC1769/GPIO13: track 46.8 -> 72.8 mm
- net /LPC1769/GPIO12: track 55.6 -> 81.4 mm
- net /LPC1769/GPIO11: track 58.2 -> 83.8 mm
- net /LPC1769/GPIO8: track 82.0 -> 105.6 mm
- net /LPC1769/GPIO7: track 84.5 -> 107.9 mm
- net /LPC1769/GPIO9: track 73.9 -> 97.1 mm
- net /LPC1769/GPIO4: track 111.6 -> 129.9 mm
- net /LPC1769/GPIO6: track 100.2 -> 116.4 mm
- net /LPC1769/GPIO5: track 102.7 -> 118.8 mm
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Other:
- outline, holes or cut-outs redrawn
- board text added: "Proyecto Final Ingeniería Electrónica R.H.O. 12-09-2016"
